File: GestureRecognition_v0.1/GestureRecognition.kicad_pcb (KiCad board)
At the start: 2 copper layers, 40 x 18 mm, 33 parts, among them U1 USB_GoldFinger, U2 ATMEGA32U4-MU, U3 SPX3819M5, U4 APDS-9960, Y1 Crystal_16M

Commit message: update
Parts:
- added G***: LOGO, OpenSourceHardware:OpenSourceHardware, B.Cu at (165.2, 102.5)
- added K1: TS-018_TS24CA, BPI:TS-018_TS24CA, B.Cu at (155.1, 90.0)
- moved C5 0.99 mm to (155.6, 92.3)
Routing:
- net GND: track 22.1 -> 29.4 mm
- net /RST: track 16.7 -> 21.9 mm
- net +5V: track 82.2 -> 79.2 mm
