File: GestureRecognition_v0.1/GestureRecognition.sch (KiCad schematic (older format))
At the start: 33 parts, among them U1 USB_GoldFinger, U2 ATMEGA32U4-MU, U3 SPX3819M5, U4 APDS-9960, Y1 Crystal_16M

Commit message: update
Parts:
- added K1: TS-018_TS24CA, BPI:TS-018_TS24CA, symbol BPI:TS-018_TS24CA
Connections:
- net GND: now also K1.1
- net RST: now also K1.2
- no-connect marks 16 -> 17
Changed lines of the file:
@@
 $EndComp
 $Comp
-L power:GND #PWR?
+L power:GND #PWR0133
 U 1 1 5E9804F4
 P 980 4970
-F 0 "#PWR?" H 980 4720 50  0001 C CNN
+F 0 "#PWR0133" H 980 4720 50  0001 C CNN
 F 1 "GND" H 985 4797 50  0000 C CNN
 F 2 "" H 980 4970 50  0001 C CNN
@@
 Wire Wire Line
 	2930 6760 2960 6760
+NoConn ~ 1230 4860
+$Comp
+L BPI:TS-018_TS24CA K1
+U 1 1 5E60D38F
+P 8800 3890
+F 0 "K1" H 8880 3840 50  0000 C CNN
+F 1 "TS-018_TS24CA" H 8857 3968 50  0001 C CNN
+F 2 "BPI:TS-018_TS24CA" H 8857 3968 50  0001 C CNN
+F 3 "" H 8857 3968 50  0001 C CNN
+	1    8800 3890
+	-1   0    0    1
+$EndComp
+$Comp
+L power:GND #PWR0142
+U 1 1 5E60E28C
+P 8900 3890
+F 0 "#PWR0142" H 8900 3640 50  0001 C CNN
+F 1 "GND" V 8905 3717 50  0000 C CNN
+F 2 "" H 8900 3890 50  0001 C CNN
+F 3 "" H 8900 3890 50  0001 C CNN
+	1    8900 3890
+	0    -1   -1   0
+$EndComp
+Wire Wire Line
+	8550 3890 8510 3890
+Wire Wire Line
+	8510 3890 8510 3700
+Connection ~ 8510 3700
 $EndSCHEMATC
